File: KiCAD/SBC80-CF.sch (KiCad schematic (older format))
At the start: 18 parts, among them J1 Conn_02x20_Odd_Even, J2 I/O ADDR JP, J3 CF Card Conn, U1 74HC138, U2 74HC04

Commit message: CFカード部品変更 REV2基板整備
Parts:
- J3: footprint Connector_Card:CF-Card_3M_N7E50-7516PK-20-WF -> Connector:CF-50P
Changed lines of the file:
@@
 F 0 "J3" H 7950 4667 50  0000 C CNN
 F 1 "CF Card Conn" H 7950 4576 50  0000 C CNN
-F 2 "Connector_Card:CF-Card_3M_N7E50-7516PK-20-WF" H 7900 3250 50  0001 C CNN
+F 2 "Connector:CF-50P" H 7900 3250 50  0001 C CNN
 F 3 "~" H 7900 3250 50  0001 C CNN
 	1    7900 3250
@@
 Wire Wire Line
 	6650 3200 7000 3200
+Connection ~ 7000 3200
+Wire Wire Line
+	7000 3200 7000 3250
 Wire Bus Line
 	2800 1750 2800 3750
@@
 Wire Bus Line
 	7300 1750 7300 4150
-Connection ~ 7000 3200
-Wire Wire Line
-	7000 3200 7000 3250
 $EndSCHEMATC
